File: BPS_Scrutineering.sch (KiCad schematic (older format))
At the start: 21 parts, among them J1 Conn_01x07_Male, J2 Conn_01x07_Male, J3 Conn_01x07_Male, J4 Conn_01x07_Male

Commit message: ready for peer review
Parts:
- R1: value R -> 0
Connections:
- net labels added: External_source
- no-connect marks 0 -> 2
Changed lines of the file:
@@
 P 2000 4650
 F 0 "R1" V 1793 4650 50  0000 C CNN
-F 1 "R" V 1884 4650 50  0000 C CNN
+F 1 "0" V 1884 4650 50  0000 C CNN
 F 2 "Resistor_SMD:R_0805_2012Metric" V 1930 4650 50  0001 C CNN
 F 3 "~" H 2000 4650 50  0001 C CNN
@@
 Wire Wire Line
 	2150 4650 2300 4650
+Wire Wire Line
+	1700 4650 1850 4650
+NoConn ~ 2900 4650
+Text Label 1250 4800 0    50   ~ 0
+External_source
+$Comp
+L power:PWR_FLAG #FLG0101
+U 1 1 5F8E9AEA
+P 1700 4650
+F 0 "#FLG0101" H 1700 4725 50  0001 C CNN
+F 1 "PWR_FLAG" H 1700 4823 50  0000 C CNN
+F 2 "" H 1700 4650 50  0001 C CNN
+F 3 "~" H 1700 4650 50  0001 C CNN
+	1    1700 4650
+	1    0    0    -1
+$EndComp
+Connection ~ 1700 4650
 $Comp
 L Device:Jumper JP16
@@
 	1    0    0    -1
 $EndComp
-Wire Wire Line
-	1700 4650 1850 4650
+NoConn ~ 1100 4650
 $EndSCHEMATC

Commit message: Add files via upload
Parts:
- added H1: MountingHole, MountingHole:MountingHole_3mm, symbol Mechanical:MountingHole
Changed lines of the file:
@@
 $EndComp
 NoConn ~ 1100 4650
+$Comp
+L Mechanical:MountingHole H1
+U 1 1 5F9473C1
+P 4400 4250
+F 0 "H1" H 4500 4296 50  0000 L CNN
+F 1 "MountingHole" H 4500 4205 50  0000 L CNN
+F 2 "MountingHole:MountingHole_3mm" H 4400 4250 50  0001 C CNN
+F 3 "~" H 4400 4250 50  0001 C CNN
+	1    4400 4250
+	1    0    0    -1
+$EndComp
 $EndSCHEMATC

Commit message: Add files via upload
Parts:
- removed JP1, JP10, JP11, JP12, JP13, JP14, JP15, JP16, JP2, JP3, JP4, JP5, JP6, JP7, JP8, JP9: Jumper, Connector_PinHeader_2.54mm:PinHeader_1x02_P2.54mm_Vertical, symbol Device:Jumper
- removed R1: 0, Resistor_SMD:R_0805_2012Metric, symbol Device:R
- added J1, J10, J11, J12, J13, J14, J2, J3, J4, J5, J6, J7, J8, J9: Conn_01x01_Female, Connector:Banana_Jack_1Pin, symbol Connector:Conn_01x01_Female
- added SW1, SW10, SW11, SW12, SW13, SW14, SW2, SW3, SW4, SW5, SW6, SW7, SW8, SW9: SW_SPST, Button_Switch_SMD:SW_SPST_B3S-1000, symbol Switch:SW_SPST
Connections:
- net labels removed: External_source
- wire segments 86 -> 119
- no-connect marks 2 -> 0

Commit message: schematic done, editing PCB, number of banana jacks?
Parts:
- removed SW1, SW10, SW11, SW12, SW13, SW14, SW2, SW3, SW4, SW5, SW6, SW7, SW8, SW9: SW_SPST, Button_Switch_SMD:SW_SPST_B3S-1000, symbol Switch:SW_SPST
- added H2, H3, H4, H5, H6: MountingHole, MountingHole:MountingHole_3mm, symbol Mechanical:MountingHole
- added SW1, SW2: SW_DIP_x07, Button_Switch_SMD:SW_DIP_SPSTx07_Slide_6.7x19.34mm_W6.73mm_P2.54mm_LowProfile_JPin, symbol Switch:SW_DIP_x07
- renumbered J1 to JC1, J2 to JC2, J3 to JC3, J4 to JC4
Connections:
- wire segments 119 -> 42
Other:
- moved on the sheet: H1, J2, J3, J4, J5, J6, J7, JC2, JC3, JC4

Commit message: Finished PCB
Parts:
- removed H1, H2, H3, H4, H5, H6: MountingHole, MountingHole:MountingHole_3mm, symbol Mechanical:MountingHole
- added LOGO1: Logo_Placeholder, UTSVT_Special:UTSVT_Logo_Symbol, symbol utsvt-misc:Logo_Placeholder
- added LOGO2: Logo_Placeholder, UTSVT_Special:Hallock_Image, symbol utsvt-misc:Logo_Placeholder
Changed lines of the file:
@@
-$EndComp
-$Comp
-L Mechanical:MountingHole H1
-U 1 1 5F9473C1
-P 4650 2000
-F 0 "H1" H 4750 2046 50  0000 L CNN
-F 1 "MountingHole" H 4750 1955 50  0000 L CNN
-F 2 "MountingHole:MountingHole_3mm" H 4650 2000 50  0001 C CNN
-F 3 "~" H 4650 2000 50  0001 C CNN
-	1    4650 2000
-	1    0    0    -1
 $EndComp
 $Comp
@@
 $EndComp
 $Comp
-L Mechanical:MountingHole H2
-U 1 1 5FAEC2DE
-P 4650 2200
-F 0 "H2" H 4750 2246 50  0000 L CNN
-F 1 "MountingHole" H 4750 2155 50  0000 L CNN
-F 2 "MountingHole:MountingHole_3mm" H 4650 2200 50  0001 C CNN
-F 3 "~" H 4650 2200 50  0001 C CNN
-	1    4650 2200
-	1    0    0    -1
-$EndComp
-$Comp
-L Mechanical:MountingHole H3
-U 1 1 5FAF0045
-P 4650 2400
-F 0 "H3" H 4750 2446 50  0000 L CNN
-F 1 "MountingHole" H 4750 2355 50  0000 L CNN
-F 2 "MountingHole:MountingHole_3mm" H 4650 2400 50  0001 C CNN
-F 3 "~" H 4650 2400 50  0001 C CNN
-	1    4650 2400
-	1    0    0    -1
-$EndComp
-$Comp
-L Mechanical:MountingHole H4
-U 1 1 5FAF40EC
-P 5400 2000
-F 0 "H4" H 5500 2046 50  0000 L CNN
-F 1 "MountingHole" H 5500 1955 50  0000 L CNN
-F 2 "MountingHole:MountingHole_3mm" H 5400 2000 50  0001 C CNN
-F 3 "~" H 5400 2000 50  0001 C CNN
-	1    5400 2000
-	1    0    0    -1
-$EndComp
-$Comp
-L Mechanical:MountingHole H5
-U 1 1 5FAF7F09
-P 5400 2200
-F 0 "H5" H 5500 2246 50  0000 L CNN
-F 1 "MountingHole" H 5500 2155 50  0000 L CNN
-F 2 "MountingHole:MountingHole_3mm" H 5400 2200 50  0001 C CNN
-F 3 "~" H 5400 2200 50  0001 C CNN
-	1    5400 2200
-	1    0    0    -1
-$EndComp
-$Comp
-L Mechanical:MountingHole H6
-U 1 1 5FAFBD75
-P 5400 2400
-F 0 "H6" H 5500 2446 50  0000 L CNN
-F 1 "MountingHole" H 5500 2355 50  0000 L CNN
-F 2 "MountingHole:MountingHole_3mm" H 5400 2400 50  0001 C CNN
-F 3 "~" H 5400 2400 50  0001 C CNN
-	1    5400 2400
-	1    0    0    -1
-$EndComp
-$Comp
 L Switch:SW_DIP_x07 SW1
 U 1 1 5FADB5F5
@@
 Wire Wire Line
 	3800 3050 3650 3050
+$Comp
+L utsvt-misc:Logo_Placeholder LOGO1
+U 1 1 5FB02C91
+P 4800 2100
+F 0 "LOGO1" H 4800 2250 50  0001 C CNN
+F 1 "Logo_Placeholder" H 4940 2100 50  0000 L CNN
+F 2 "UTSVT_Special:UTSVT_Logo_Symbol" H 4800 2175 50  0001 C CNN
+F 3 "" H 4800 2175 50  0001 C CNN
+	1    4800 2100
+	1    0    0    -1
+$EndComp
+$Comp
+L utsvt-misc:Logo_Placeholder LOGO2
+U 1 1 5FB04696
+P 4800 1500
+F 0 "LOGO2" H 4800 1650 50  0001 C CNN
+F 1 "Logo_Placeholder" H 4940 1500 50  0000 L CNN
+F 2 "UTSVT_Special:Hallock_Image" H 4800 1575 50  0001 C CNN
+F 3 "" H 4800 1575 50  0001 C CNN
+	1    4800 1500
+	1    0    0    -1
+$EndComp
 $EndSCHEMATC

Commit message: Flipped Connectors
Parts:
- JC1, JC2, JC3, JC4: value Conn_01x07_Male -> Conn_01x07; footprint Connector_PinHeader_2.54mm:PinHeader_1x07_P2.54mm_Vertical -> Connector_Molex:Molex_Micro-Fit_3.0_43650-0700_1x07_P3.00mm_Horizontal; symbol Connector:Conn_01x07_Male -> Connector_Generic:Conn_01x07
- renumbered LOGO2 to Dr_Hallock1, LOGO1 to UTSVT_Logo1
Changed lines of the file:
@@
 $EndDescr
 $Comp
-L Connector:Conn_01x07_Male JC4
+L Connector_Generic:Conn_01x07 JC4
 U 1 1 5F94FA02
-P 1400 2750
-F 0 "JC4" H 1508 3231 50  0000 C CNN
-F 1 "Conn_01x07_Male" H 1508 3140 50  0000 C CNN
-F 2 "Connector_PinHeader_2.54mm:PinHeader_1x07_P2.54mm_Vertical" H 1400 2750 50  0001 C CNN
-F 3 "~" H 1400 2750 50  0001 C CNN
-	1    1400 2750
-	1    0    0    -1
-$EndComp
-$Comp
-L Connector:Conn_01x07_Male JC2
+P 1450 2750
+F 0 "JC4" H 1558 3231 50  0000 C CNN
+F 1 "Conn_01x07" H 1558 3140 50  0000 C CNN
+F 2 "Connector_Molex:Molex_Micro-Fit_3.0_43650-0700_1x07_P3.00mm_Horizontal" H 1450 2750 50  0001 C CNN
+F 3 "~" H 1450 2750 50  0001 C CNN
+	1    1450 2750
+	1    0    0    -1
+$EndComp
+$Comp
+L Connector_Generic:Conn_01x07 JC2
 U 1 1 5F9521B3
-P 4000 1700
-F 0 "JC2" H 3972 1632 50  0000 R CNN
-F 1 "Conn_01x07_Male" H 3972 1723 50  0000 R CNN
-F 2 "Connector_PinHeader_2.54mm:PinHeader_1x07_P2.54mm_Vertical" H 4000 1700 50  0001 C CNN
-F 3 "~" H 4000 1700 50  0001 C CNN
-	1    4000 1700
+P 3950 1700
+F 0 "JC2" H 3922 1632 50  0000 R CNN
+F 1 "Conn_01x07" V 3922 1723 50  0000 R CNN
+F 2 "Connector_Molex:Molex_Micro-Fit_3.0_43650-0700_1x07_P3.00mm_Horizontal" H 3950 1700 50  0001 C CNN
+F 3 "~" H 3950 1700 50  0001 C CNN
+	1    3950 1700
 	-1   0    0    1
 $EndComp
@@
 $EndComp
 $Comp
-L Connector:Conn_01x07_Male JC3
+L Connector_Generic:Conn_01x07 JC3
 U 1 1 5F9537A8
-P 4000 2750
-F 0 "JC3" H 3972 2682 50  0000 R CNN
-F 1 "Conn_01x07_Male" H 3972 2773 50  0000 R CNN
-F 2 "Connector_PinHeader_2.54mm:PinHeader_1x07_P2.54mm_Vertical" H 4000 2750 50  0001 C CNN
-F 3 "~" H 4000 2750 50  0001 C CNN
-	1    4000 2750
+P 3950 2750
+F 0 "JC3" H 3922 2682 50  0000 R CNN
+F 1 "Conn_01x07" H 3922 2773 50  0000 R CNN
+F 2 "Connector_Molex:Molex_Micro-Fit_3.0_43650-0700_1x07_P3.00mm_Horizontal" H 3950 2750 50  0001 C CNN
+F 3 "~" H 3950 2750 50  0001 C CNN
+	1    3950 2750
 	-1   0    0    1
 $EndComp
@@
 $EndComp
 $Comp
-L Connector:Conn_01x07_Male JC1
+L Connector_Generic:Conn_01x07 JC1
 U 1 1 5F94EF32
-P 1400 1700
-F 0 "JC1" H 1508 2181 50  0000 C CNN
-F 1 "Conn_01x07_Male" H 1508 2090 50  0000 C CNN
-F 2 "Connector_PinHeader_2.54mm:PinHeader_1x07_P2.54mm_Vertical" H 1400 1700 50  0001 C CNN
-F 3 "~" H 1400 1700 50  0001 C CNN
-	1    1400 1700
+P 1450 1700
+F 0 "JC1" H 1558 2181 50  0000 C CNN
+F 1 "Conn_01x07" H 1558 2090 50  0000 C CNN
+F 2 "Connector_Molex:Molex_Micro-Fit_3.0_43650-0700_1x07_P3.00mm_Horizontal" H 1450 1700 50  0001 C CNN
+F 3 "~" H 1450 1700 50  0001 C CNN
+	1    1450 1700
 	1    0    0    -1
 $EndComp
@@
 $EndComp
 Wire Wire Line
-	1600 1400 2550 1400
-Wire Wire Line
-	1600 1500 2550 1500
-Wire Wire Line
-	1600 1600 2550 1600
-Wire Wire Line
-	1600 1700 2550 1700
-Wire Wire Line
-	2550 1800 1600 1800
-Wire Wire Line
-	1600 1900 2550 1900
-Wire Wire Line
-	2550 2000 1600 2000
-Wire Wire Line
 	2550 1400 3050 1400
 Connection ~ 2550 1400
 Wire Wire Line
 	3050 1500 2550 1500
-Connection ~ 2550 1500
 Wire Wire Line
 	3050 1600 2550 1600
@@
 	3050 2000 2550 2000
 Connection ~ 2550 2000
-Wire Wire Line
-	3650 1400 3800 1400
-Wire Wire Line
-	3800 1500 3650 1500
-Wire Wire Line
-	3800 1600 3650 1600
-Wire Wire Line
-	3800 1700 3650 1700
-Wire Wire Line
-	3800 1800 3650 1800
-Wire Wire Line
-	3800 1900 3650 1900
-Wire Wire Line
-	3800 2000 3650 2000
 $Comp
 L Connector:Conn_01x01_Female J9
@@
 $EndComp
 Wire Wire Line
-	1600 2450 2550 2450
-Wire Wire Line
-	1600 2550 2550 2550
-Wire Wire Line
-	1600 2650 2550 2650
-Wire Wire Line
-	1600 2750 2550 2750
-Wire Wire Line
-	2550 2850 1600 2850
-Wire Wire Line
-	1600 2950 2550 2950
-Wire Wire Line
-	2550 3050 1600 3050
-Wire Wire Line
 	2550 2450 3050 2450
 Connection ~ 2550 2450
 Wire Wire Line
 	3050 2550 2550 2550
-Connection ~ 2550 2550
 Wire Wire Line
 	3050 2650 2550 2650
@@
 	3050 3050 2550 3050
 Connection ~ 2550 3050
-Wire Wire Line
-	3650 2450 3800 2450
-Wire Wire Line
-	3800 2550 3650 2550
-Wire Wire Line
-	3800 2650 3650 2650
-Wire Wire Line
-	3800 2750 3650 2750
-Wire Wire Line
-	3800 2850 3650 2850
-Wire Wire Line
-	3800 2950 3650 2950
-Wire Wire Line
-	3800 3050 3650 3050
-$Comp
-L utsvt-misc:Logo_Placeholder LOGO1
+$Comp
+L utsvt-misc:Logo_Placeholder UTSVT_Logo1
 U 1 1 5FB02C91
 P 4800 2100
-F 0 "LOGO1" H 4800 2250 50  0001 C CNN
+F 0 "UTSVT_Logo1" H 4800 2250 50  0001 C CNN
 F 1 "Logo_Placeholder" H 4940 2100 50  0000 L CNN
 F 2 "UTSVT_Special:UTSVT_Logo_Symbol" H 4800 2175 50  0001 C CNN
@@
 $EndComp
 $Comp
-L utsvt-misc:Logo_Placeholder LOGO2
+L utsvt-misc:Logo_Placeholder Dr_Hallock1
 U 1 1 5FB04696
 P 4800 1500
-F 0 "LOGO2" H 4800 1650 50  0001 C CNN
+F 0 "Dr_Hallock1" H 4800 1650 50  0001 C CNN
 F 1 "Logo_Placeholder" H 4940 1500 50  0000 L CNN
 F 2 "UTSVT_Special:Hallock_Image" H 4800 1575 50  0001 C CNN
@@
 	1    0    0    -1
 $EndComp
+Connection ~ 2550 1500
+Connection ~ 2550 2550
+Wire Wire Line
+	1250 1400 2550 1400
+Wire Wire Line
+	1250 1500 2550 1500
+Wire Wire Line
+	1250 1900 2550 1900
+Wire Wire Line
+	1250 2000 2550 2000
+Wire Wire Line
+	1250 1800 2550 1800
+Wire Wire Line
+	1250 1600 2550 1600
+Wire Wire Line
+	1250 1700 2550 1700
+Wire Wire Line
+	3650 1400 4150 1400
+Wire Wire Line
+	3650 1500 4150 1500
+Wire Wire Line
+	3650 1600 4150 1600
+Wire Wire Line
+	3650 1700 4150 1700
+Wire Wire Line
+	3650 1800 4150 1800
+Wire Wire Line
+	3650 1900 4150 1900
+Wire Wire Line
+	3650 2000 4150 2000
+Wire Wire Line
+	3650 2450 4150 2450
+Wire Wire Line
+	3650 2550 4150 2550
+Wire Wire Line
+	3650 2650 4150 2650
+Wire Wire Line
+	3650 2750 4150 2750
+Wire Wire Line
+	3650 2850 4150 2850
+Wire Wire Line
+	3650 2950 4150 2950
+Wire Wire Line
+	3650 3050 4150 3050
+Wire Wire Line
+	1250 2450 2550 2450
+Wire Wire Line
+	1250 2550 2550 2550
+Wire Wire Line
+	1250 2650 2550 2650
+Wire Wire Line
+	1250 2750 2550 2750
+Wire Wire Line
+	1250 2850 2550 2850
+Wire Wire Line
+	1250 2950 2550 2950
+Wire Wire Line
+	1250 3050 2550 3050
 $EndSCHEMATC

Commit message: Changed footprints
Parts:
- J1, J10, J11, J12, J13, J14, J2, J3, J4, J5, J6, J7, J8, J9: footprint Connector:Banana_Jack_1Pin -> UTSVT_Connectors:Banana_Jack_1_Pin_4mm
Changed lines of the file:
@@
 F 0 "J2" H 2778 1526 50  0000 L CNN
 F 1 "Conn_01x01_Female" H 1850 1550 50  0000 L CNN
-F 2 "Connector:Banana_Jack_1Pin" H 2750 1500 50  0001 C CNN
+F 2 "UTSVT_Connectors:Banana_Jack_1_Pin_4mm" H 2750 1500 50  0001 C CNN
 F 3 "~" H 2750 1500 50  0001 C CNN
 	1    2750 1500
@@
 F 0 "J3" H 2778 1626 50  0000 L CNN
 F 1 "Conn_01x01_Female" H 1850 1650 50  0000 L CNN
-F 2 "Connector:Banana_Jack_1Pin" H 2750 1600 50  0001 C CNN
+F 2 "UTSVT_Connectors:Banana_Jack_1_Pin_4mm" H 2750 1600 50  0001 C CNN
 F 3 "~" H 2750 1600 50  0001 C CNN
 	1    2750 1600
@@
 F 0 "J5" H 2778 1826 50  0000 L CNN
 F 1 "Conn_01x01_Female" H 1850 1850 50  0000 L CNN
-F 2 "Connector:Banana_Jack_1Pin" H 2750 1800 50  0001 C CNN
+F 2 "UTSVT_Connectors:Banana_Jack_1_Pin_4mm" H 2750 1800 50  0001 C CNN
 F 3 "~" H 2750 1800 50  0001 C CNN
 	1    2750 1800
@@
 F 0 "J6" H 2778 1926 50  0000 L CNN
 F 1 "Conn_01x01_Female" H 1850 1950 50  0000 L CNN
-F 2 "Connector:Banana_Jack_1Pin" H 2750 1900 50  0001 C CNN
+F 2 "UTSVT_Connectors:Banana_Jack_1_Pin_4mm" H 2750 1900 50  0001 C CNN
 F 3 "~" H 2750 1900 50  0001 C CNN
 	1    2750 1900
@@
 F 0 "J7" H 2778 2026 50  0000 L CNN
 F 1 "Conn_01x01_Female" H 1850 2050 50  0000 L CNN
-F 2 "Connector:Banana_Jack_1Pin" H 2750 2000 50  0001 C CNN
+F 2 "UTSVT_Connectors:Banana_Jack_1_Pin_4mm" H 2750 2000 50  0001 C CNN
 F 3 "~" H 2750 2000 50  0001 C CNN
 	1    2750 2000
@@
 F 0 "J1" H 2778 1426 50  0000 L CNN
 F 1 "Conn_01x01_Female" H 1850 1450 50  0000 L CNN
-F 2 "Connector:Banana_Jack_1Pin" H 2750 1400 50  0001 C CNN
+F 2 "UTSVT_Connectors:Banana_Jack_1_Pin_4mm" H 2750 1400 50  0001 C CNN
 F 3 "~" H 2750 1400 50  0001 C CNN
 	1    2750 1400
@@
 F 0 "J4" H 2778 1726 50  0000 L CNN
 F 1 "Conn_01x01_Female" H 1850 1750 50  0000 L CNN
-F 2 "Connector:Banana_Jack_1Pin" H 2750 1700 50  0001 C CNN
+F 2 "UTSVT_Connectors:Banana_Jack_1_Pin_4mm" H 2750 1700 50  0001 C CNN
 F 3 "~" H 2750 1700 50  0001 C CNN
 	1    2750 1700
@@
 F 0 "J9" H 2778 2576 50  0000 L CNN
 F 1 "Conn_01x01_Female" H 1850 2600 50  0000 L CNN
-F 2 "Connector:Banana_Jack_1Pin" H 2750 2550 50  0001 C CNN
+F 2 "UTSVT_Connectors:Banana_Jack_1_Pin_4mm" H 2750 2550 50  0001 C CNN
 F 3 "~" H 2750 2550 50  0001 C CNN
 	1    2750 2550
@@
 F 0 "J10" H 2778 2676 50  0000 L CNN
 F 1 "Conn_01x01_Female" H 1850 2700 50  0000 L CNN
-F 2 "Connector:Banana_Jack_1Pin" H 2750 2650 50  0001 C CNN
+F 2 "UTSVT_Connectors:Banana_Jack_1_Pin_4mm" H 2750 2650 50  0001 C CNN
 F 3 "~" H 2750 2650 50  0001 C CNN
 	1    2750 2650
@@
 F 0 "J12" H 2778 2876 50  0000 L CNN
 F 1 "Conn_01x01_Female" H 1850 2900 50  0000 L CNN
-F 2 "Connector:Banana_Jack_1Pin" H 2750 2850 50  0001 C CNN
+F 2 "UTSVT_Connectors:Banana_Jack_1_Pin_4mm" H 2750 2850 50  0001 C CNN
 F 3 "~" H 2750 2850 50  0001 C CNN
 	1    2750 2850
@@
 F 0 "J13" H 2778 2976 50  0000 L CNN
 F 1 "Conn_01x01_Female" H 1850 3000 50  0000 L CNN
-F 2 "Connector:Banana_Jack_1Pin" H 2750 2950 50  0001 C CNN
+F 2 "UTSVT_Connectors:Banana_Jack_1_Pin_4mm" H 2750 2950 50  0001 C CNN
 F 3 "~" H 2750 2950 50  0001 C CNN
 	1    2750 2950
@@
 F 0 "J14" H 2778 3076 50  0000 L CNN
 F 1 "Conn_01x01_Female" H 1850 3100 50  0000 L CNN
-F 2 "Connector:Banana_Jack_1Pin" H 2750 3050 50  0001 C CNN
+F 2 "UTSVT_Connectors:Banana_Jack_1_Pin_4mm" H 2750 3050 50  0001 C CNN
 F 3 "~" H 2750 3050 50  0001 C CNN
 	1    2750 3050
@@
 F 0 "J8" H 2778 2476 50  0000 L CNN
 F 1 "Conn_01x01_Female" H 1850 2500 50  0000 L CNN
-F 2 "Connector:Banana_Jack_1Pin" H 2750 2450 50  0001 C CNN
+F 2 "UTSVT_Connectors:Banana_Jack_1_Pin_4mm" H 2750 2450 50  0001 C CNN
 F 3 "~" H 2750 2450 50  0001 C CNN
 	1    2750 2450
@@
 F 0 "J11" H 2778 2776 50  0000 L CNN
 F 1 "Conn_01x01_Female" H 1850 2800 50  0000 L CNN
-F 2 "Connector:Banana_Jack_1Pin" H 2750 2750 50  0001 C CNN
+F 2 "UTSVT_Connectors:Banana_Jack_1_Pin_4mm" H 2750 2750 50  0001 C CNN
 F 3 "~" H 2750 2750 50  0001 C CNN
 	1    2750 2750
