File: BPS_Scrutineering.kicad_sch (KiCad schematic)
At the start: 54 parts, among them SW1 SW_DIP_x07, SW2 SW_DIP_x07

Commit message: Finished Schematic
Parts:
- removed Dr_Hallock1: Dr. Hallock, UTSVT_Special:Hallock_Image, symbol utsvt-misc:Logo_Placeholder
- removed F1, F15, F22, F8: PTC Fuse, UTSVT_Special:ptc_fuse_FUSC1607X75N, symbol Device:Polyfuse_Small
- removed F10, F11, F12, F13, F14, F16, F17, F18, F19, F2, F20, F21, F23, F24, F25, F26, F27, F28, F3, F4, F5, F6, F7, F9: PTC_Fuse, UTSVT_Special:ptc_fuse_FUSC1607X75N, symbol Device:Polyfuse_Small
- removed H1, H2, H3, H4: MountingHole, MountingHole:MountingHole_3mm_Pad, symbol Mechanical:MountingHole
- removed JC1, JC2, JC3, JC4: Conn_01x07, UTSVT_Connectors:Molex_Microfit+_01x07_Horizontal, symbol Connector_Generic:Conn_01x07
- removed SW1, SW2: SW_DIP_x07, UTSVT_Special:7switch_module_DS04254207BKSMT, symbol Switch:SW_DIP_x07
- removed TP1, TP10, TP11, TP12, TP13, TP14, TP2, TP3, TP4, TP5, TP6, TP7, TP8, TP9: TestPoint, TestPoint:TestPoint_Keystone_5005-5009_Compact, symbol Connector:TestPoint
- removed UTSVT_Logo1: UTSVT, UTSVT_Special:UTSVT_Logo_Symbol, symbol utsvt-misc:Logo_Placeholder
Connections:
- no-connect marks 0 -> 7
Other:
- added sheet BATT_SEG_1 (battery_interface.kicad_sch)
- added sheet BATT_SEG_2 (battery_interface.kicad_sch)
- added sheet BATT_SEG_3 (battery_interface.kicad_sch)
- added sheet BATT_SEG_4 (battery_interface.kicad_sch)
- added sheet BPS_MINION_1 (minion_interface.kicad_sch)
- added sheet BPS_MINION_2 (minion_interface.kicad_sch)
- added sheet BPS_MINION_3 (minion_interface.kicad_sch)
- added sheet DIP_SW_1 (dip_interface.kicad_sch)
- added sheet DIP_SW_2 (dip_interface.kicad_sch)
- added sheet DIP_SW_3 (dip_interface.kicad_sch)
- added sheet DIP_SW_4 (dip_interface.kicad_sch)
- added sheet DIP_SW_5 (dip_interface.kicad_sch)
- added sheet DIP_SW_6 (dip_interface.kicad_sch)
- note removed: "Battery Module Side"
- note removed: "Minion Board Side"
